Commit message: modify

File: sim1_lecture/urdf/arm_robot.urdf (robot description, URDF)
Before this commit: robot arm_robot, 3 links, 2 joints
Links:
- link arm1_link: mass 1.0 -> 0.1
- link base_link: mass 1.0 -> 0.1

File: sim2_lecture/xacro/dtw_camera.xacro (robot description, xacro)
@@ -11,4 +11,6 @@
     <plugin name="gazebo_ros_control" filename="libgazebo_ros_control.so">
       <robotNamespace>/dtw_robot</robotNamespace>
+      <robotSimType>gazebo_ros_control/DefaultRobotHWSim</robotSimType>
+      <legacyModeNS>true</legacyModeNS>
     </plugin>
   </gazebo>

File: sim2_lecture/xacro/dtw_imu.xacro (robot description, xacro)
@@ -11,4 +11,6 @@
     <plugin name="gazebo_ros_control" filename="libgazebo_ros_control.so">
       <robotNamespace>/dtw_robot</robotNamespace>
+      <robotSimType>gazebo_ros_control/DefaultRobotHWSim</robotSimType>
+      <legacyModeNS>true</legacyModeNS>
     </plugin>
   </gazebo>

File: sim2_lecture/xacro/dtw_laser.xacro (robot description, xacro)
@@ -11,4 +11,6 @@
     <plugin name="gazebo_ros_control" filename="libgazebo_ros_control.so">
       <robotNamespace>/dtw_robot</robotNamespace>
+      <robotSimType>gazebo_ros_control/DefaultRobotHWSim</robotSimType>
+      <legacyModeNS>true</legacyModeNS>
     </plugin>
   </gazebo>

File: sim2_lecture/xacro/dtw_move_only.xacro (robot description, xacro)
@@ -9,4 +9,6 @@
     <plugin name="gazebo_ros_control" filename="libgazebo_ros_control.so">
       <robotNamespace>/dtw_robot</robotNamespace>
+      <robotSimType>gazebo_ros_control/DefaultRobotHWSim</robotSimType>
+      <legacyModeNS>true</legacyModeNS>
     </plugin>
   </gazebo>

File: sim2_lecture/xacro/odm_single_wheel_only.xacro (robot description, xacro)
@@ -8,4 +8,6 @@
     <plugin name="gazebo_ros_control" filename="libgazebo_ros_control.so">
       <robotNamespace>/odm_robot</robotNamespace>
+      <robotSimType>gazebo_ros_control/DefaultRobotHWSim</robotSimType>
+      <legacyModeNS>true</legacyModeNS>
     </plugin>
   </gazebo>

File: sim2_lecture/xacro/odm_try_wheel1.xacro (robot description, xacro)
@@ -50,4 +50,6 @@
     <plugin name="gazebo_ros_control" filename="libgazebo_ros_control.so">
       <robotNamespace>/odm_robot</robotNamespace>
+      <robotSimType>gazebo_ros_control/DefaultRobotHWSim</robotSimType>
+      <legacyModeNS>true</legacyModeNS>
     </plugin>
   </gazebo>

File: sim2_lecture/xacro/odm_try_wheel2.xacro (robot description, xacro)
@@ -50,4 +50,6 @@
     <plugin name="gazebo_ros_control" filename="libgazebo_ros_control.so">
       <robotNamespace>/odm_robot</robotNamespace>
+      <robotSimType>gazebo_ros_control/DefaultRobotHWSim</robotSimType>
+      <legacyModeNS>true</legacyModeNS>
     </plugin>
   </gazebo>
