Commit message: gazebo2_lecture: update

File: gazebo2_lecture/urdf/wheel_robot_sensor.urdf (robot description, URDF)
Before this commit: robot dtw_robot, 6 links, 5 joints
Links:
- added link depth_camera_link
- added link head_camera_link
- added link left_back_sonar_link
- added link right_back_sonar_link
Joints:
- added joint depth_camera_joint: type fixed, parent body_link, child depth_camera_link, origin xyz=0 0 0.15 rpy=-1.5707 0 -1.5707
- added joint head_camera_joint: type fixed, parent body_link, child head_camera_link, origin xyz=0 0 0.15 rpy=-1.5707 0 -1.5707
- added joint left_back_sonar_joint: type fixed, parent body_link, child left_back_sonar_link, origin xyz=-0.27 0.17 0 rpy=0 0 2.97
- added joint right_back_sonar_joint: type fixed, parent body_link, child right_back_sonar_link, origin xyz=-0.27 -0.17 0 rpy=0 0 -2.97

Commit message: update

File: gazebo2_lecture/urdf/wheel_robot_sensor.urdf (robot description, URDF)
Before this commit: robot dtw_robot, 10 links, 9 joints
Links:
- added link main_imu_link
Joints:
- added joint main_imu_joint: type fixed, parent body_link, child main_imu_link, origin xyz=-0.10 0 0.15 rpy=0 0 0
