Commit message: modify nav_lecture

File: nav_lecture/xacro/dtw_robot.xacro (robot description, xacro)
@@ -11,5 +11,5 @@
   <xacro:wheel_macro prefix="left_wheel"  parent="base_link" xyz="0 0.1 0.05"/>
   <xacro:wheel_macro prefix="right_wheel" parent="base_link" xyz="0 -0.1 0.05"/>
-  <xacro:laser_macro prefix="front_laser" parent="base_link" xyz="0 0 0.13" />
+  <xacro:laser_macro prefix="front_laser" parent="base_link" xyz="0 0 0.13" robot_name="$(arg robot_name)"/>
   <xacro:imu_macro prefix="imu" parent="base_link" xyz="-0.05 0 0.10" robot_name="$(arg robot_name)"/>
   <xacro:camera_macro prefix="head_camera" parent="base_link" xyz="0.1 0 0.08"/>

File: nav_lecture/xacro/laser_macro.xacro (robot description, xacro)
@@ -1,5 +1,5 @@
 <?xml version="1.0"?>
 <robot name="dtw_robot" xmlns:xacro="http://ros.org/wiki/xacro">
-  <xacro:macro name="laser_macro" params="parent prefix xyz">
+  <xacro:macro name="laser_macro" params="parent prefix xyz robot_name">
     <joint name="${prefix}_joint" type="fixed">
       <parent link="${parent}"/>
@@ -50,5 +50,5 @@
         <plugin name="gazebo_ros_lidar_controller" filename="libgazebo_ros_laser.so">
           <topicName>${prefix}/scan</topicName>
-          <frameName>${prefix}_link</frameName>
+          <frameName>${robot_name}/${prefix}_link</frameName>
         </plugin>
       </sensor>
